File: cad/brain_pcb/arachne_brain.kicad_pcb (KiCad board)
At the start: 4 copper layers, 140 x 70 mm, 114 parts, among them J1 12V IN, J10 FAN, J11 PI LINK, J2 L1 servo, J3 L2 servo, J4 L3 servo, J5 L4 servo, J6 L5 servo, J7 L6 servo, J8 USB-C ESP32, J9 USB-C CM5, M1 CM5 (wireless), Q1 AOD4185, Q2 2N7002, Q3 2N7002, Q4 2N7002, Q5 2N7002, SW1 RESET, SW2 BOOT, SW3 RPIBOOT, SW4 AAN/UIT, U1 TPS54560B, U10 USBLC6-2SC6, U11 FSUSB42MUX, U12 USBLC6-2SC6, U2 AMS1117-3.3, U3 ESP32-S3-WROOM-1-N16R8, U4 74AHCT1G126, U5 74LVC1G34, U6 74AHCT1G126, U7 74LVC1G34, U8 MPU-6050, U9 74LVC1G34

Commit message: Name Kobe Vanrobaeys on silkscreen/schematic, fresh JLC fab files for brain_mini
Co-Authored-By: Claude Opus 5.5 <noreply@anthropic.com>
Other:
- board text added: "Kobe Vanrobaeys · maakleerplek · 2026"
- board text removed: "Kobe Van Robaeys · maakleerplek · 2026"
Changed lines of the file:
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@@
 			)
 		)
-		(attr smd dnp)
+		(attr smd)
 		(duplicate_pad_numbers_are_jumpers no)
 		(fp_line
@@
 			)
 		)
-		(attr smd dnp)
+		(attr smd)
 		(duplicate_pad_numbers_are_jumpers no)
 		(fp_line
@@
 			)
 		)
-		(attr smd dnp)
+		(attr smd)
 		(duplicate_pad_numbers_are_jumpers no)
 		(fp_line
@@
 			)
 		)
-		(attr smd dnp)
+		(attr smd)
 		(duplicate_pad_numbers_are_jumpers no)
 		(fp_line
@@
 			)
 		)
-		(attr smd dnp)
+		(attr smd)
 		(duplicate_pad_numbers_are_jumpers no)
 		(fp_line
@@
 			)
 		)
-		(attr smd dnp)
+		(attr smd)
 		(duplicate_pad_numbers_are_jumpers no)
 		(fp_line
@@
 			)
 		)
-		(attr smd dnp)
+		(attr smd)
 		(duplicate_pad_numbers_are_jumpers no)
 		(fp_line
@@
 			)
 		)
-		(attr smd dnp)
+		(attr smd)
 		(duplicate_pad_numbers_are_jumpers no)
 		(fp_line
@@
 			)
 		)
-		(attr smd dnp)
+		(attr smd)
 		(duplicate_pad_numbers_are_jumpers no)
 		(fp_line
@@
 			)
 		)
-		(attr smd dnp)
+		(attr smd)
 		(duplicate_pad_numbers_are_jumpers no)
 		(fp_line
@@
 			)
 		)
-		(attr smd dnp)
+		(attr smd)
 		(duplicate_pad_numbers_are_jumpers no)
 		(fp_line
@@
 			)
 		)
-		(attr smd dnp)
+		(attr smd)
 		(duplicate_pad_numbers_are_jumpers no)
 		(fp_line
@@
 			)
 		)
-		(attr smd dnp)
+		(attr smd)
 		(duplicate_pad_numbers_are_jumpers no)
 		(fp_line
@@
 			)
 		)
-		(attr smd dnp)
+		(attr smd)
 		(duplicate_pad_numbers_are_jumpers no)
 		(fp_line
@@
 			)
 		)
-		(attr smd dnp)
+		(attr smd)
 		(duplicate_pad_numbers_are_jumpers no)
 		(fp_line
@@
 			)
 		)
-		(attr smd dnp)
+		(attr smd)
 		(duplicate_pad_numbers_are_jumpers no)
 		(fp_line
@@
 			)
 		)
-		(attr smd dnp)
+		(attr smd)
 		(duplicate_pad_numbers_are_jumpers no)
 		(fp_line
@@
 			)
 		)
-		(attr smd dnp)
+		(attr smd)
 		(duplicate_pad_numbers_are_jumpers no)
 		(fp_line
@@
 			)
 		)
-		(attr smd dnp)
+		(attr smd)
 		(duplicate_pad_numbers_are_jumpers no)
 		(fp_line
@@
 			)
 		)
-		(attr smd dnp)
+		(attr smd)
 		(duplicate_pad_numbers_are_jumpers no)
 		(fp_line
@@
 		)
 	)
-	(gr_text "Kobe Van Robaeys  ·  maakleerplek  ·  2026"
+	(gr_text "Kobe Vanrobaeys  ·  maakleerplek  ·  2026"
 		(at 150 112 0)
 		(layer "B.SilkS")
