File: cad/brain_pcb/arachne_brain.kicad_sch (KiCad schematic)
At the start: 114 parts, among them J1 12V IN, J10 FAN, J11 PI LINK, J2 L1 servo, J3 L2 servo, J4 L3 servo, J5 L4 servo, J6 L5 servo, J7 L6 servo, J8 USB-C ESP32, J9 USB-C CM5, M1 CM5 (wireless), Q1 AOD4185, Q2 2N7002, Q3 2N7002, Q4 2N7002, Q5 2N7002, SW1 RESET, SW2 BOOT, SW3 RPIBOOT, SW4 AAN/UIT, U1 TPS54560B, U10 USBLC6-2SC6, U11 FSUSB42MUX, U12 USBLC6-2SC6, U2 AMS1117-3.3, U3 ESP32-S3-WROOM-1-N16R8, U4 74AHCT1G126, U5 74LVC1G34, U6 74AHCT1G126, U7 74LVC1G34, U8 MPU-6050, U9 74LVC1G34

Commit message: Name Kobe Vanrobaeys on silkscreen/schematic, fresh JLC fab files for brain_mini
Co-Authored-By: Claude Opus 5.5 <noreply@anthropic.com>
Other:
- company: Kobe Van Robaeys - maakleerplek -> Kobe Vanrobaeys - maakleerplek
Changed lines of the file:
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@@
 		(date "2026-10-17")
 		(rev "1.0")
-		(company "Kobe Van Robaeys - maakleerplek")
+		(company "Kobe Vanrobaeys - maakleerplek")
 		(comment 1 "CM5 + ESP32-S3 + MPU-6050, 6 servo-bus legs")
 	)
