File: cad/brain_mini/arachne_mini.kicad_sch (KiCad schematic)
At the start: 89 parts, among them J1 12V IN, J13 5V PI, J14 SENSOR S, J15 SENSOR V, J16 SENSOR G, J17 I2C, J18 I2C, J2 L1 servo, J3 L2 servo, J4 L3 servo, J5 L4 servo, J6 L5 servo, J7 L6 servo, J8 USB-C PI, Q1 AOD4185, SW1 RESET, SW2 BOOT, U1 TPS54560B, U10 USBLC6-2SC6, U2 AMS1117-3.3, U3 ESP32-S3-WROOM-1-N16R8, U4 74AHCT1G126, U5 74LVC1G34, U6 74AHCT1G126, U7 74LVC1G34, U8 LSM6DS3TR-C

Commit message: JLC: every part placed again (no DNP), CPL positions = pad-field centre from the board (fixes USB-C/headers/connectors offset)
Co-Authored-By: Claude Opus 5.5 <noreply@anthropic.com>
Parts:
- C1, C2: MPN hand-solder (not placed by JLC): 330uF 25V 8x10.5 alu, STRO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 -> 330uF 25V 8x10.5 alu, STRONGLY recommended for the servo cu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; now fitted
- D1: MPN hand-solder (not placed by JLC): SMBJ15CA TVS (optional) -> SMBJ15CA TVS (optional); now fitted
- D2: MPN hand-solder (not placed by JLC): BZT52C15 gate clamp (optio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 -> BZT52C15 gate clamp (optional: AOD4185 Vgs max 20 V); now fitted
- J14: MPN hand-solder (not placed by JLC): 1x19 pin header 2.54 mm (r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 -> 1x19 pin header 2.54 mm (row S of the sensor strip); now fitted
- J15: MPN hand-solder (not placed by JLC): 1x19 pin header 2.54 mm (r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 -> 1x19 pin header 2.54 mm (row V of the sensor strip); now fitted
- J16: MPN hand-solder (not placed by JLC): 1x19 pin header 2.54 mm (r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 -> 1x19 pin header 2.54 mm (row G of the sensor strip); now fitted
- J17, J18: MPN hand-solder (not placed by JLC): JST SM04B-SRSS-TB (Qwiic /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 -> JST SM04B-SRSS-TB (Qwiic / STEMMA QT, optional); now fitted
- J2, J3, J4, J5, J6, J7: MPN hand-solder (not placed by JLC): Molex 22-03-5035 / 5267-03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 -> Molex 22-03-5035 / 5267-03A Mini-SPOX (mates with the 5264 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; now fitted
- SW1, SW2: MPN hand-solder (not placed by JLC): CK KMR221G (4.2x2.8 tact);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 -> CK KMR221G (4.2x2.8 tact); the S3 flashes over native USB w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; now fitted
- U10: MPN hand-solder (not placed by JLC): USBLC6-2SC6 ESD (optional) -> USBLC6-2SC6 ESD (optional); now fitted
Changed lines of the file:
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@@
 		(in_bom yes)
 		(on_board yes)
-		(dnp yes)
+		(dnp no)
 		(property "Reference" "D2"
 			(at 86.36 29.25 0)
@@
 			)
 		)
-		(property "MPN" "hand-solder (not placed by JLC): BZT52C15 gate clamp (optional: AOD4185 Vgs max 20 V)"
+		(property "MPN" "BZT52C15 gate clamp (optional: AOD4185 Vgs max 20 V)"
 			(at 86.36 33.02 0)
 			(effects
@@
 		(in_bom yes)
 		(on_board yes)
-		(dnp yes)
+		(dnp no)
 		(property "Reference" "D1"
 			(at 116.84 29.25 0)
@@
 			)
 		)
-		(property "MPN" "hand-solder (not placed by JLC): SMBJ15CA TVS (optional)"
+		(property "MPN" "SMBJ15CA TVS (optional)"
 			(at 116.84 33.02 0)
 			(effects
@@
 		(in_bom yes)
 		(on_board yes)
-		(dnp yes)
+		(dnp no)
 		(property "Reference" "C1"
 			(at 134.62 36.87 0)
@@
 			)
 		)
-		(property "MPN" "hand-solder (not placed by JLC): 330uF 25V 8x10.5 alu, STRONGLY recommended for the servo current peaks"
+		(property "MPN" "330uF 25V 8x10.5 alu, STRONGLY recommended for the servo current peaks"
 			(at 134.62 43.18 0)
 			(effects
@@
 		(in_bom yes)
 		(on_board yes)
-		(dnp yes)
+		(dnp no)
 		(property "Reference" "C2"
 			(at 147.32 36.87 0)
@@
 			)
 		)
-		(property "MPN" "hand-solder (not placed by JLC): 330uF 25V 8x10.5 alu, STRONGLY recommended for the servo current peaks"
+		(property "MPN" "330uF 25V 8x10.5 alu, STRONGLY recommended for the servo current peaks"
 			(at 147.32 43.18 0)
 			(effects
@@
 		(in_bom yes)
 		(on_board yes)
-		(dnp yes)
+		(dnp no)
 		(property "Reference" "SW1"
 			(at 33.02 324.652 0)
@@
 			)
 		)
-		(property "MPN" "hand-solder (not placed by JLC): CK KMR221G (4.2x2.8 tact); the S3 flashes over native USB without it"
+		(property "MPN" "CK KMR221G (4.2x2.8 tact); the S3 flashes over native USB without it"
 			(at 33.02 330.2 0)
 			(effects
@@
 		(in_bom yes)
 		(on_board yes)
-		(dnp yes)
+		(dnp no)
 		(property "Reference" "SW2"
 			(at 66.04 324.652 0)
@@
 			)
 		)
-		(property "MPN" "hand-solder (not placed by JLC): CK KMR221G (4.2x2.8 tact); the S3 flashes over native USB without it"
+		(property "MPN" "CK KMR221G (4.2x2.8 tact); the S3 flashes over native USB without it"
 			(at 66.04 330.2 0)
 			(effects
@@
 		(in_bom yes)
 		(on_board yes)
-		(dnp yes)
+		(dnp no)
 		(property "Reference" "J2"
 			(at 33.02 397.55 0)
@@
 			)
 		)
-		(property "MPN" "hand-solder (not placed by JLC): Molex 22-03-5035 / 5267-03A Mini-SPOX (mates with the 5264 plug on Feetech cables), LCSC C45581067"
+		(property "MPN" "Molex 22-03-5035 / 5267-03A Mini-SPOX (mates with the 5264 plug on Feetech cables), LCSC C45581067"
 			(at 33.02 403.86 0)
 			(effects
@@
 		(in_bom yes)
 		(on_board yes)
-		(dnp yes)
+		(dnp no)
 		(property "Reference" "J3"
 			(at 53.34 397.55 0)
@@
 			)
 		)
-		(property "MPN" "hand-solder (not placed by JLC): Molex 22-03-5035 / 5267-03A Mini-SPOX (mates with the 5264 plug on Feetech cables), LCSC C45581067"
+		(property "MPN" "Molex 22-03-5035 / 5267-03A Mini-SPOX (mates with the 5264 plug on Feetech cables), LCSC C45581067"
 			(at 53.34 403.86 0)
 			(effects
@@
 		(in_bom yes)
 		(on_board yes)
-		(dnp yes)
+		(dnp no)
 		(property "Reference" "J4"
 			(at 76.2 397.55 0)
@@
 			)
 		)
-		(property "MPN" "hand-solder (not placed by JLC): Molex 22-03-5035 / 5267-03A Mini-SPOX (mates with the 5264 plug on Feetech cables), LCSC C45581067"
+		(property "MPN" "Molex 22-03-5035 / 5267-03A Mini-SPOX (mates with the 5264 plug on Feetech cables), LCSC C45581067"
 			(at 76.2 403.86 0)
 			(effects
@@
 		(in_bom yes)
 		(on_board yes)
-		(dnp yes)
+		(dnp no)
 		(property "Reference" "J5"
 			(at 33.02 476.29 0)
@@
 			)
 		)
-		(property "MPN" "hand-solder (not placed by JLC): Molex 22-03-5035 / 5267-03A Mini-SPOX (mates with the 5264 plug on Feetech cables), LCSC C45581067"
+		(property "MPN" "Molex 22-03-5035 / 5267-03A Mini-SPOX (mates with the 5264 plug on Feetech cables), LCSC C45581067"
 			(at 33.02 482.6 0)
 			(effects
@@
 		(in_bom yes)
 		(on_board yes)
-		(dnp yes)
+		(dnp no)
 		(property "Reference" "J6"
 			(at 53.34 476.29 0)
@@
 			)
 		)
-		(property "MPN" "hand-solder (not placed by JLC): Molex 22-03-5035 / 5267-03A Mini-SPOX (mates with the 5264 plug on Feetech cables), LCSC C45581067"
+		(property "MPN" "Molex 22-03-5035 / 5267-03A Mini-SPOX (mates with the 5264 plug on Feetech cables), LCSC C45581067"
 			(at 53.34 482.6 0)
 			(effects
@@
 		(in_bom yes)
 		(on_board yes)
-		(dnp yes)
+		(dnp no)
 		(property "Reference" "J7"
 			(at 76.2 476.29 0)
@@
 			)
 		)
-		(property "MPN" "hand-solder (not placed by JLC): Molex 22-03-5035 / 5267-03A Mini-SPOX (mates with the 5264 plug on Feetech cables), LCSC C45581067"
+		(property "MPN" "Molex 22-03-5035 / 5267-03A Mini-SPOX (mates with the 5264 plug on Feetech cables), LCSC C45581067"
 			(at 76.2 482.6 0)
 			(effects
@@
 		(in_bom yes)
 		(on_board yes)
-		(dnp yes)
+		(dnp no)
 		(property "Reference" "U10"
 			(at 287.02 106.72 0)
@@
 			)
 		)
-		(property "MPN" "hand-solder (not placed by JLC): USBLC6-2SC6 ESD (optional)"
+		(property "MPN" "USBLC6-2SC6 ESD (optional)"
 			(at 287.02 114.3 0)
 			(effects
@@
 		(in_bom yes)
 		(on_board yes)
-		(dnp yes)
+		(dnp no)
 		(property "Reference" "J14"
 			(at 220.98 184.19 0)
@@
 			)
 		)
-		(property "MPN" "hand-solder (not placed by JLC): 1x19 pin header 2.54 mm (row S of the sensor strip)"
+		(property "MPN" "1x19 pin header 2.54 mm (row S of the sensor strip)"
 			(at 220.98 210.82 0)
 			(effects
@@
 		(in_bom yes)
 		(on_board yes)
-		(dnp yes)
+		(dnp no)
 		(property "Reference" "J15"
 			(at 241.3 184.19 0)
@@
 			)
 		)
-		(property "MPN" "hand-solder (not placed by JLC): 1x19 pin header 2.54 mm (row V of the sensor strip)"
+		(property "MPN" "1x19 pin header 2.54 mm (row V of the sensor strip)"
 			(at 241.3 210.82 0)
 			(effects
@@
 		(in_bom yes)
 		(on_board yes)
-		(dnp yes)
+		(dnp no)
 		(property "Reference" "J16"
 			(at 261.62 184.19 0)
@@
 			)
 		)
-		(property "MPN" "hand-solder (not placed by JLC): 1x19 pin header 2.54 mm (row G of the sensor strip)"
+		(property "MPN" "1x19 pin header 2.54 mm (row G of the sensor strip)"
 			(at 261.62 210.82 0)
 			(effects
@@
 		(in_bom yes)
 		(on_board yes)
-		(dnp yes)
+		(dnp no)
 		(property "Reference" "J17"
 			(at 284.48 189.27 0)
@@
 			)
 		)
-		(property "MPN" "hand-solder (not placed by JLC): JST SM04B-SRSS-TB (Qwiic / STEMMA QT, optional)"
+		(property "MPN" "JST SM04B-SRSS-TB (Qwiic / STEMMA QT, optional)"
 			(at 284.48 195.58 0)
 			(effects
@@
 		(in_bom yes)
 		(on_board yes)
-		(dnp yes)
+		(dnp no)
 		(property "Reference" "J18"
 			(at 309.88 189.27 0)
@@
 			)
 		)
-		(property "MPN" "hand-solder (not placed by JLC): JST SM04B-SRSS-TB (Qwiic / STEMMA QT, optional)"
+		(property "MPN" "JST SM04B-SRSS-TB (Qwiic / STEMMA QT, optional)"
 			(at 309.88 195.58 0)
 			(effects

Commit message: JLC: sensor headers J14-J16 hand-soldered (DNP), TO-252 rotation +180
Co-Authored-By: Claude Opus 5.5 <noreply@anthropic.com>
Parts:
- J14: MPN 1x19 pin header 2.54 mm (row S of the sensor strip) -> 1x19 pin header 2.54 mm (row S of the sensor strip), hand-s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; now not fitted
- J15: MPN 1x19 pin header 2.54 mm (row V of the sensor strip) -> 1x19 pin header 2.54 mm (row V of the sensor strip), hand-s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; now not fitted
- J16: MPN 1x19 pin header 2.54 mm (row G of the sensor strip) -> 1x19 pin header 2.54 mm (row G of the sensor strip), hand-s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; now not fitted
Changed lines of the file:
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@@
 		(in_bom yes)
 		(on_board yes)
-		(dnp no)
+		(dnp yes)
 		(property "Reference" "J14"
 			(at 220.98 184.19 0)
@@
 			)
 		)
-		(property "MPN" "1x19 pin header 2.54 mm (row S of the sensor strip)"
+		(property "MPN" "1x19 pin header 2.54 mm (row S of the sensor strip), hand-soldered"
 			(at 220.98 210.82 0)
 			(effects
@@
 		(in_bom yes)
 		(on_board yes)
-		(dnp no)
+		(dnp yes)
 		(property "Reference" "J15"
 			(at 241.3 184.19 0)
@@
 			)
 		)
-		(property "MPN" "1x19 pin header 2.54 mm (row V of the sensor strip)"
+		(property "MPN" "1x19 pin header 2.54 mm (row V of the sensor strip), hand-soldered"
 			(at 241.3 210.82 0)
 			(effects
@@
 		(in_bom yes)
 		(on_board yes)
-		(dnp no)
+		(dnp yes)
 		(property "Reference" "J16"
 			(at 261.62 184.19 0)
@@
 			)
 		)
-		(property "MPN" "1x19 pin header 2.54 mm (row G of the sensor strip)"
+		(property "MPN" "1x19 pin header 2.54 mm (row G of the sensor strip), hand-soldered"
 			(at 261.62 210.82 0)
 			(effects
